File: hardware/improved-handheld-turbidimeter_TIA.brd (EAGLE design)
At the start: 23 x 17.8 mm, 13 parts

Commit message: updates to TIA
Routing:
- net N$1: track 9.26 -> 12.6 mm
- net GND: track 0.00 -> 2.08 mm, vias 0 -> 1
Other:
- board text added: "AWQUA TIA Board v1.1 2016/10/27"
- board text removed: "AWQUA TIA Board v1.0 2016/08/24"
Changed lines of the file:
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@@
 <?xml version="1.0" encoding="utf-8"?>
 <!DOCTYPE eagle SYSTEM "eagle.dtd">
-<eagle version="7.6.0">
+<eagle version="7.3.0">
 <drawing>
 <settings>
@@
 <text x="18.123" y="4.332" size="1.27" layer="26" rot="MR0">AWQUA
 TIA Board
-v1.0
-2016/08/24</text>
+v1.1
+2016/10/27</text>
 <text x="14.986" y="1.905" size="1.524" layer="25">+</text>
 <text x="8.255" y="1.778" size="2.032" layer="25">-</text>
@@
 <contactref element="JP3" pad="2"/>
 <polygon width="0.254" layer="16">
-<vertex x="-2.54" y="21.336"/>
+<vertex x="-2.286" y="20.828"/>
 <vertex x="25.908" y="21.082"/>
 <vertex x="25.654" y="-2.794"/>
-<vertex x="-1.27" y="-1.27"/>
+<vertex x="-2.667" y="-3.048"/>
 </polygon>
 <polygon width="0.254" layer="1">
@@
 </polygon>
 <contactref element="U$2" pad="P$4"/>
+<wire x1="9.627" y1="9.48" x2="9.627" y2="8.534" width="0.254" layer="1"/>
+<wire x1="9.627" y1="8.534" x2="9.779" y2="8.382" width="0.254" layer="1"/>
+<wire x1="9.779" y1="8.382" x2="10.287" y2="7.62" width="0.254" layer="1"/>
+<via x="10.287" y="7.62" extent="1-16" drill="0.6" shape="square"/>
 </signal>
 <signal name="OUTA">
@@
 <contactref element="PDA_RF" pad="1"/>
 <contactref element="PDA" pad="1"/>
-<wire x1="2.54" y1="6.858" x2="2.54" y2="9.017" width="0.254" layer="1"/>
-<wire x1="2.54" y1="9.017" x2="1.905" y2="9.652" width="0.254" layer="1"/>
-<wire x1="1.905" y1="9.652" x2="1.905" y2="11.518" width="0.254" layer="1"/>
-<wire x1="1.905" y1="11.518" x2="3.175" y2="12.788" width="0.254" layer="1"/>
 <wire x1="3.175" y1="12.788" x2="5.715" y2="12.788" width="0.254" layer="1"/>
+<wire x1="2.54" y1="6.858" x2="2.54" y2="7.747" width="0.254" layer="1"/>
+<wire x1="2.54" y1="7.747" x2="1.27" y2="9.017" width="0.254" layer="1"/>
+<wire x1="1.27" y1="9.017" x2="1.27" y2="13.208" width="0.254" layer="1"/>
+<wire x1="1.27" y1="13.208" x2="2.032" y2="13.97" width="0.254" layer="1"/>
+<wire x1="2.032" y1="13.97" x2="2.667" y2="13.97" width="0.254" layer="1"/>
+<wire x1="2.667" y1="13.97" x2="3.302" y2="13.335" width="0.254" layer="1"/>
+<wire x1="3.302" y1="13.335" x2="3.302" y2="12.915" width="0.254" layer="1"/>
+<wire x1="3.302" y1="12.915" x2="3.175" y2="12.788" width="0.254" layer="1"/>
 </signal>
 <signal name="N$2">
@@
 <wire x1="16.695" y1="10.13" x2="17.653" y2="11.088" width="0.254" layer="1"/>
 </signal>
-<signal name="N$7">
-<via x="10.414" y="7.62" extent="1-16" drill="0.3302" shape="square"/>
-</signal>
 <signal name="N$8">
